File: docs/research/fixtures/atomfab-kicad-cli-smoke/continuity-coupon.kicad_pcb (KiCad board)
At the start: 2 copper layers, 20 x 13 mm, 2 parts, among them J1 CONTINUITY, J2 CONTINUITY

Commit message: fix(atomfab): make smoke coupon footprints self-contained
Parts:
- J1: footprint Connector_PinHeader_2.54mm:PinHeader_1x02_P2.54mm_Vertical -> AtomFab_Continuity_Connector_VCC
- J2: footprint Connector_PinHeader_2.54mm:PinHeader_1x02_P2.54mm_Vertical -> AtomFab_Continuity_Connector_GND
Changed lines of the file:
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@@
     (add_net "GND")
   )
-  (footprint "Connector_PinHeader_2.54mm:PinHeader_1x02_P2.54mm_Vertical"
+  (footprint "AtomFab_Continuity_Connector_VCC"
     (layer "F.Cu")
     (at 105 100)
@@
     )
   )
-  (footprint "Connector_PinHeader_2.54mm:PinHeader_1x02_P2.54mm_Vertical"
+  (footprint "AtomFab_Continuity_Connector_GND"
     (layer "F.Cu")
     (at 115 100)
